File: schemat/naswietlarka.brd (EAGLE design)
At the start: 95.2 x 69.5 mm, 31 parts, among them IC2 MEGA8-P, K1 G5L, T1 BC547, T2 BC547, T3 BC547

Commit message: poprawiona wersja schematu i płytki
Parts:
- removed DIS1: TUXGR_16X2_R2, display-lcd:TUXGR_16X2_R2
- removed JP2, JP3, JP4: (no value), pinhead:1X02
- removed JP5: (no value), pinhead:1X04
- removed LED_GREEN, LED_RED: (no value), led:LED5MM
- removed T1, T2, T3: BC547, transistor:TO92
- removed U$2: (no value), synergia_logo:SYNERGIA_20MM
- removed X6: (no value), con-ptr500:AK500/3-H
- added C1, C3, C4, C5: 100n, rcl:C0805
- added C2, C6, C7: 47u, rcl:E2,5-5
- added D1: 1N4148DO35-7, diode:DO35-7
- added IC1: 7805TV, linear:TO220V
- added Q1, Q2: BSS123, transistor-small-signal:SOT23
- added SV1: (no value), con-harting-ml:ML14
- DOWN, OK, RESET, UP: value 9077-1 -> (none); device switch-misc:9077-1 -> con-ptr500:AK300/2
- F1: value (none) -> 250mA
- F2: value (none) -> 500mA
- JP1: device pinhead:1X02 -> pinhead:1X03
- KRANC, KRANC.BEZP: value 9077-1 -> (none); device switch-misc:9077-1 -> con-ptr500:AK300/3
- R1: value (none) -> 10k
- U$1: device synergia_logo:SYNERGIA_20MM -> synergia_logo:SYNERGIA_30MM
- moved R1 47.5 mm to (15.2, 71.1)
- moved KRANC.BEZP 43.3 mm to (77.5, 14.0)
- moved KRANC 36.1 mm to (15.2, 14.0), turned to 0 degrees
- moved RESET 35.6 mm to (63.5, 14.0), turned to 0 degrees
- moved JP1 34.0 mm to (16.5, 30.8), turned to 270 degrees
- moved X1 32.2 mm to (52.1, 28.3)
- moved DOWN 25.5 mm to (40.6, 14.0)
- moved F2 24.2 mm to (58.4, 39.4), turned to 180 degrees
- moved SG1 22.9 mm to (26.7, 71.1), turned to 270 degrees
- moved UP 21.6 mm to (29.2, 14.0), turned to 0 degrees
- moved OK 17.1 mm to (52.1, 14.0), turned to 0 degrees
- moved IC2 15.2 mm to (48.3, 53.3)
- moved U$1 6.84 mm to (86.4, 25.4), flipped to the top
- moved X5 4.58 mm to (62.2, 72.4)
- moved X4 4.02 mm to (50.8, 72.4)
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Connections:
- removed net AVCC: IC2.20
- removed net EN_PWM: IC2.14, T3.2
- removed net LED_GREEN: IC2.28, LED_GREEN.A
- removed net LED_RED: IC2.27, LED_RED.A
- removed net N$7: DIS1.2
- removed net N$9: T3.3, X6.1
- new net VSS: K1.O, X2.2, X3.2, X4.2, X5.2
- net +5V: now also C1.2, C2.+, C4.2, C5.2, C6.+, D1.C, IC1.3, IC2.20, JP1.2, KRANC.1, KRANC.BEZP.1, SV1.12, SV1.2; no longer F2.2, JP4.1, JP5.3, KRANC.3, KRANC.BEZP.3, X6.3
- net BUZZER: now also IC2.14, Q1.1; no longer IC2.12, T2.2
- net GND: now also C1.1, C2.-, C3.1, C4.1, C5.1, C6.-, C7.-, IC1.2, JP1.3, KRANC.3, KRANC.BEZP.3, Q1.2, Q2.2, SV1.1, SV1.11, SV1.4; no longer JP4.2, JP5.1, JP5.4, K1.O, KRANC.1, KRANC.BEZP.1, LED_GREEN.K, LED_RED.K, T1.1, T2.1, T3.1, X2.2, X3.2, X4.2, X5.2
- net N$1: now also R1.A, SV1.3; no longer JP5.2, R1.E
- net N$2: now also D1.A, Q2.3; no longer T1.3
- net N$4: now also Q1.3; no longer T2.3
- net N$6: now also C3.2, C7.+, F2.2, IC1.1; no longer DIS1.1
- net PB2: now also SV1.5; no longer JP3.2
- net PB3: now also SV1.6; no longer JP3.1
- net PB4: now also SV1.7; no longer JP2.2
- net PB5: now also SV1.8; no longer JP2.1
- net PB6: now also SV1.9; no longer JP1.2
- net PB7: now also SV1.10; no longer JP1.1
- net PWM: now also JP1.1; no longer X6.2
- net RELAY: now also Q2.1; no longer T1.2
Routing:
- net GND: track 30.0 -> 380.2 mm, vias 6 -> 0
- net +5V: track 159.8 -> 348.2 mm, vias 0 -> 4
- net VSS: track 0.00 -> 138.0 mm
- net UV: track 133.8 -> 54.9 mm
- net KRANC.BEZP: track 7.87 -> 77.0 mm
- net KRANC: track 11.7 -> 73.7 mm
- net PB6: track 7.40 -> 64.0 mm, vias 0 -> 2
- net PB4: track 7.62 -> 52.3 mm
- net RESET: track 8.64 -> 51.8 mm
- net PB2: track 7.62 -> 50.0 mm
- net UP: track 20.4 -> 58.6 mm
- net PB7: track 7.40 -> 43.3 mm, vias 0 -> 2
- net RELAY: track 24.0 -> 53.8 mm, vias 0 -> 2
- net PB5: track 7.62 -> 36.1 mm, vias 0 -> 2
- net EN_PWM: track 27.8 -> 0.00 mm
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- added copper zone on layer 1, net GND
Other:
- board size 95.2 x 69.5 mm -> 109.2 x 79.7 mm
- board text added: "-5V+"
- board text added: "DOWN"
- board text added: "J. Trzyna"
- board text added: "KRANC"
- board text added: "OK"
- board text added: "RST"
- board text added: "SERWO"
- board text added: "UP"
- board text added: "UV lamps"
- board text added: "kranc. bezp"
- board text removed: "1"
- board text removed: "11"
- board text removed: "12"
- board text removed: "13"
- board text removed: "14"
- board text removed: "15"
- board text removed: "16"
- board text removed: "2"
- board text removed: "3"
- board text removed: "4"
- board text removed: "5"
- board text removed: "5V"
- board text removed: "6"
- board text removed: "UV"
- board text removed: "buzz"
- board text removed: "dow"
- board text removed: "kr"
- board text removed: "kr.b"
- board text removed: "led"
- board text removed: "ok"
- board text removed: "rst"
- board text removed: "serwo"
- board text removed: "up"
- board text removed: "uv"
