File: schemat/naswietlarka.sch (EAGLE design)
At the start: 21 parts, among them IC2 MEGA8-P, K1 G5L, T1 BC547, T2 BC547

Commit message: jazda 1.5s do przodu i powrot, ilosc petli konfigurowalna
Parts:
- added F2: (no value), fuse:SH22,5
- added JP1, JP2, JP3, JP4: (no value), pinhead:PINHD-1X2
- added JP5: (no value), pinhead:PINHD-1X4
- added T3: BC547, transistor:BC547
- added X6: (no value), con-ptr500:AK500/3-H
- DOWN, KRANC, KRANC.BEZP, OK, RESET, UP: value 9450-1 -> 9077-1; device switch-misc:9450-1 -> switch-misc:9077-1
- R1: value 2k2 -> (none); device rcl:R-EU_0207/15 -> pot:TRIM_EU-CA6V
Connections:
- new net EN_PWM: IC2.PB0(ICP), T3.B
- new net N$5: F2.1, X1-1.KL
- new net N$6: DIS1.GND
- new net N$7: DIS1.VCC
- new net N$9: T3.C, X6-1.KL
- net +5V: now also F2.2, JP4.1, JP5.3, X6-3.KL; no longer DIS1.NC@2, DOWN.O, OK.O, RESET.O, UP.O, X1-1.KL
- net BUZZER: now also IC2.PD6(AIN0); no longer IC2.PB0(ICP)
- net GND: now also JP4.2, JP5.1, JP5.4, R1.S, T3.E; no longer DIS1.GND, DIS1.NC@1, DIS1.R/W, R1.2
- net N$1: now also JP5.2, R1.E; no longer DIS1.CONTR, R1.1
- net PB2: now also IC2.PB2(SS/OC1B), JP3.2; no longer DIS1.RS
- net PB3: now also JP3.1; no longer DIS1.E
- net PB4: now also JP2.2; no longer DIS1.D4
- net PB5: now also JP2.1; no longer DIS1.D5
- net PB6: now also JP1.2; no longer DIS1.D6
- net PB7: now also JP1.1; no longer DIS1.D7
- net PWM: now also X6-2.KL
- net VCC: no longer DIS1.VCC
Other:
- note added: "Serwo"
- moved on the sheet: DOWN, KRANC, KRANC.BEZP, OK, RESET, UP

Commit message: poprawiona wersja schematu i płytki
Parts:
- removed DIS1: TUXGR_16X2_R2, display-lcd:TUXGR_16X2_R2
- removed JP2, JP3, JP4: (no value), pinhead:PINHD-1X2
- removed JP5: (no value), pinhead:PINHD-1X4
- removed LED_GREEN, LED_RED: (no value), led:LED5MM
- removed T1, T2, T3: BC547, transistor:BC547
- removed X6: (no value), con-ptr500:AK500/3-H
- added C1, C3, C4, C5: 100n, rcl:C-EUC0805
- added C2, C6, C7: 47u, rcl:CPOL-EUE2.5-5
- added D1: 1N4148DO35-7, diode:1N4148DO35-7
- added IC1: 7805TV, linear:7805TV
- added Q1, Q2: BSS123, transistor-small-signal:BSS123
- added SV1: (no value), con-harting-ml:ML14
- DOWN, OK, RESET, UP: value 9077-1 -> (none); device switch-misc:9077-1 -> con-ptr500:AK300/2
- F1: value (none) -> 250mA
- F2: value (none) -> 500mA
- JP1: device pinhead:PINHD-1X2 -> pinhead:PINHD-1X3
- KRANC, KRANC.BEZP: value 9077-1 -> (none); device switch-misc:9077-1 -> con-ptr500:AK300/3
- R1: value (none) -> 10k
Connections:
- removed net EN_PWM: IC2.PB0(ICP), T3.B
- removed net LED_GREEN: IC2.PC5(ADC5/SCL), LED_GREEN.A
- removed net LED_RED: IC2.PC4(ADC4/SDA), LED_RED.A
- removed net N$7: DIS1.VCC
- removed net N$9: T3.C, X6-1.KL
- new net VSS: K12.O, X2-2.KL, X3-2.KL, X4-2.KL, X5-2.KL
- net +5V: now also C1.2, C2.+, C4.2, C5.2, C6.+, D1.C, IC1.VO, IC2.AVCC, JP1.2, KRANC-1.KL, KRANC.BEZP-1.KL, SV1.12, SV1.2; no longer F2.2, JP4.1, JP5.3, KRANC.BEZP.O, KRANC.O, X6-3.KL
- net BUZZER: now also IC2.PB0(ICP), Q1.G; no longer IC2.PD6(AIN0), T2.B
- net DOWN: now also DOWN-2.KL; no longer DOWN.P
- net GND: now also C1.1, C2.-, C3.1, C4.1, C5.1, C6.-, C7.-, DOWN-1.KL, IC1.GND, IC2.GND, JP1.3, KRANC-3.KL, KRANC.BEZP-3.KL, OK-1.KL, Q1.S, Q2.S, RESET-1.KL, SV1.1, SV1.11, SV1.4, UP-1.KL; no longer DOWN.S, JP4.2, JP5.1, JP5.4, K12.O, KRANC.BEZP.S, KRANC.S, LED_GREEN.C, LED_RED.C, OK.S, RESET.S, T1.E, T2.E, T3.E, UP.S, X2-2.KL, X3-2.KL, X4-2.KL, X5-2.KL
- net KRANC: now also KRANC-2.KL; no longer KRANC.P
- net KRANC.BEZP: now also KRANC.BEZP-2.KL; no longer KRANC.BEZP.P
- net N$1: now also R1.A, SV1.3; no longer JP5.2, R1.E
- net N$2: now also D1.A, Q2.D; no longer T1.C
- net N$4: now also Q1.D; no longer T2.C
- net N$6: now also C3.2, C7.+, F2.2, IC1.VI; no longer DIS1.GND
- net OK: now also OK-2.KL; no longer OK.P
- net PB2: now also SV1.5; no longer JP3.2
- net PB3: now also SV1.6; no longer JP3.1
- net PB4: now also SV1.7; no longer JP2.2
- net PB5: now also SV1.8; no longer JP2.1
- net PB6: now also SV1.9; no longer JP1.2
- net PB7: now also SV1.10; no longer JP1.1
- net PWM: now also JP1.1; no longer X6-2.KL
- net RELAY: now also Q2.G; no longer T1.B
- net RESET: now also RESET-2.KL; no longer RESET.P
- net UP: now also UP-2.KL; no longer UP.P
Other:
- note added: "1 - GND 2 - +5V 3 - POT 4 - PB2 5 - GND 6 - PB3 11 - PB4 12 - PB5 13 - PB6 14 - PB7 15 - GND 16 - +5V"
- note removed: "LEDs"
- moved on the sheet: F1, F2, R1, X1-1, X1-2, X2-1, X2-2
